File: DC34-Mech-SAO/DC34-Mech-SAO.kicad_sch (KiCad schematic)
At the start: 20 parts, among them J1 Conn_01x06_Male, J2 Conn_01x03_Male, U1 ATtiny816-M

Commit message: change_3
added laser cannon
Connections:
- net +3.3V: now also R5.2
- net GND: no longer R5.2
