File: DC34-Mech-SAO/DC34-Mech-SAO.kicad_pcb (KiCad board)
At the start: 2 copper layers, 27.9 x 38 mm, 20 parts, among them J1 Conn_01x06_Male, J2 Conn_01x03_Male, U1 ATtiny816-M

Commit message: Updated Traces for Design Rule Check
Made it so that power and ground traces do not violate design rule checks.
Routing:
- net GND: track 115.9 -> 117.7 mm
- net PWR: track 87.2 -> 88.5 mm
